Commit message: Added hands and fingers

File: v1/urdf/v1.urdf (robot description, URDF)
Before this commit: robot v1, 21 links, 20 joints
Links:
- added link LLFingerL, mass 0.00367689699109765; collision mesh filename=package://v1/meshes/LLFingerL.STL; visual mesh filename=package://v1/meshes/LLFingerL.STL
- added link LLFingerU, mass 0.0104365547026631; collision mesh filename=package://v1/meshes/LLFingerU.STL; visual mesh filename=package://v1/meshes/LLFingerU.STL
- added link LPalm, mass 0.071951528369027; collision mesh filename=package://v1/meshes/LPalm.STL; visual mesh filename=package://v1/meshes/LPalm.STL
- added link LRFingerL, mass 0.00367689699109764; collision mesh filename=package://v1/meshes/LRFingerL.STL; visual mesh filename=package://v1/meshes/LRFingerL.STL
- added link LRFingerU, mass 0.0104365547041236; collision mesh filename=package://v1/meshes/LRFingerU.STL; visual mesh filename=package://v1/meshes/LRFingerU.STL
- added link LWrist, mass 0.0707291405501728; collision mesh filename=package://v1/meshes/LWrist.STL; visual mesh filename=package://v1/meshes/LWrist.STL
- added link RLFingerL, mass 0.00367689699109765; collision mesh filename=package://v1/meshes/RLFingerL.STL; visual mesh filename=package://v1/meshes/RLFingerL.STL
- added link RLFingerU, mass 0.0104365547181582; collision mesh filename=package://v1/meshes/RLFingerU.STL; visual mesh filename=package://v1/meshes/RLFingerU.STL
- added link RPalm, mass 0.0719515165156188; collision mesh filename=package://v1/meshes/RPalm.STL; visual mesh filename=package://v1/meshes/RPalm.STL
- added link RRFingerL, mass 0.00367689699109764; collision mesh filename=package://v1/meshes/RRFingerL.STL; visual mesh filename=package://v1/meshes/RRFingerL.STL
- added link RRFingerU, mass 0.0104365547185436; collision mesh filename=package://v1/meshes/RRFingerU.STL; visual mesh filename=package://v1/meshes/RRFingerU.STL
- added link RWrist, mass 0.0707291283778046; collision mesh filename=package://v1/meshes/RWrist.STL; visual mesh filename=package://v1/meshes/RWrist.STL
- link LLFemur: mass 0.0813765964956518 -> 0.0813765964956519
- link LLHumerus: mass 0.0924406077669575 -> 0.0924406076207102
- link LRadius: mass 0.225239496648543 -> 0.225239465270569
- link RFoot: mass 0.0576266868508424 -> 0.0576266868508423
- link RLFemur: mass 0.0813765923276173 -> 0.0813766060772551
- link RMFemur: mass 0.123790789571376 -> 0.123790727728343
- link RTibia: mass 0.197322267255763 -> 0.197322298408282
- link RToe: mass 0.0300993542432527 -> 0.0300993381405375
- link RUFemur: mass 0.0588371617715196 -> 0.0588371599148218
Joints:
- added joint LLKnuckleL: type continuous, parent LLFingerU, child LLFingerL, origin xyz=-0.0230295534577176 0.00418692684763539 0.00654490271930316 rpy=0 0 -1.39256651875685, axis 0 0 1
- added joint LLKnuckleU: type continuous, parent LPalm, child LLFingerU, origin xyz=1.84275573584247E-05 -0.0513442857142855 0 rpy=0 0 0.0795874815148373, axis 0 0 1
- added joint LRKnuckleL: type continuous, parent LRFingerU, child LRFingerL, origin xyz=-0.0330185105270897 -0.00134428488911487 0.00626872193397954 rpy=0 0 -1.33697789041426, axis 0 0 1
- added joint LRKnuckleU: type continuous, parent LPalm, child LRFingerU, origin xyz=1.84275573584247E-05 -0.05 0.000276180785323571 rpy=0 0 -0.00110800345436074, axis 0 0 1
- added joint LWrist1: type continuous, parent LRadius, child LWrist, origin xyz=0 -0.154047567567568 0 rpy=1.57079632679489 -1.56895051945567 -1.57079632679489, axis 0 0 1
- added joint LWrist2: type continuous, parent LWrist, child LPalm, origin xyz=0 0 0 rpy=0 -0.0666240559322892 0, axis 0 1 0
- added joint RLKnuckleL: type continuous, parent RLFingerU, child RLFingerL, origin xyz=-0.0330199999999999 0 -0.00815796517422882 rpy=0 0 -1.42852646400694, axis 0 0 1
- added joint RLKnuckleU: type continuous, parent RPalm, child RLFingerU, origin xyz=0 -0.0513442857142855 0.000962687485064811 rpy=0 0 0.0322968189623831, axis 0 0 1
- added joint RRKnuckleL: type continuous, parent RRFingerU, child RRFingerL, origin xyz=-0.0329799188990406 -0.00134368805419179 0.00680985742226439 rpy=0 0 -1.42676533867921, axis 0 0 1
- added joint RRKnuckleU: type continuous, parent RPalm, child RRFingerU, origin xyz=0 -0.05 0.000276725129630978 rpy=0 0 -0.0298203287563768, axis 0 0 1
- added joint RWrist1: type continuous, parent RRadius, child RWrist, origin xyz=0 -0.154047567567566 0 rpy=-1.5707963267949 0.763601167462532 -1.5707963267949, axis 0 0 1
- added joint RWrist2: type continuous, parent RWrist, child RPalm, origin xyz=0 0 0 rpy=0 -0.0224487832351522 0, axis 0 1 0
- joint LAnkle: origin xyz=0 -0.139583099293917 0.00131428947187286 rpy=-1.5707963267949 -1.48050713192401 1.5707963267949 -> xyz=0 -0.137327472527473 0 rpy=-1.5707963267949 -1.48050713192401 1.5707963267949
- joint LElbow1: origin xyz=0 -0.0608622763001231 0 rpy=-3.14159265358979 0.169197756118627 3.14159265358979 -> xyz=0 -0.0607173844560569 0 rpy=-3.14159265358979 -0.0239343941798154 3.14159265358979
- joint LElbow2: origin xyz=0 -0.0768125885647418 0 rpy=2.6860465798041 0 -3.14159265358979 -> xyz=0 -0.07695748040881 0 rpy=-3.03329101627937 0 -3.14159265358979
- joint LKnee1: origin xyz=0 -0.0702723715213309 0 rpy=0 -0.21670904669546 0 -> xyz=-0.250689445253999 -0.0779374608440729 0.210317560896771 rpy=0 -0.21670904669546 0
- joint LKnee2: origin xyz=0 -0.05 0 rpy=0.527580516456534 0 0 -> xyz=0.1790209512322 -0.0449455061888935 -0.259300751969874 rpy=0.527580516456534 0 0
- joint RAnkle: origin xyz=0 -0.141066763777475 0.00190498731071205 rpy=1.57079632679491 -1.22947386247953 -1.57079632679491 -> xyz=0 -0.136901508135358 -0.000553841883564526 rpy=-1.5707963267949 -1.19317274042075 1.5707963267949
- joint RElbow2: origin xyz=0 -0.0899704517869545 0 rpy=0.613164267402606 0 0 -> xyz=0 -0.0899704517869562 0 rpy=0.441432869104159 0 0
- joint RHip1: origin xyz=0.03048 -0.0787364118309958 0.0381 rpy=-1.63511592849543 0 -1.5707963267949 -> xyz=0.03048 -0.0787364118309958 0.0380999999999998 rpy=-1.76467257912073 0 -1.5707963267949
- joint RHip2: origin xyz=0.0226409652141426 0.0442211339031965 0.00572015878352808 rpy=-0.128639141191749 0.000126862066806489 -3.1406119141409 -> xyz=0.0226409652141427 0.0412792847511113 0.0168597019733423 rpy=-0.386092293810914 -0.0367782603560909 3.05138185304591
- joint RKnee1: origin xyz=0 -0.0686863879849429 0 rpy=0 -0.029939106057863 0 -> xyz=0 -0.073581670471731 0 rpy=0 -0.221518435550964 0
- joint RKnee2: origin xyz=0 -0.05 0 rpy=0.471180140436868 0 0 -> xyz=0 -0.05 0 rpy=0.915177643816393 0 0
- joint RToe: origin xyz=0.05000625 0 0 rpy=0 0 0.465479513878318 -> xyz=0.05000625 0 0 rpy=0 0 -0.000476651083853421

Commit message: fixed joint zero positions

File: v1/urdf/v1.urdf (robot description, URDF)
Before this commit: robot v1, 33 links, 32 joints
Links:
- link LLFemur: mass 0.0813765964956519 -> 0.0813765868175624
- link LLFingerL: mass 0.00367689699109765 -> 0.00367689699109764
- link LLFingerU: mass 0.0104365547026631 -> 0.0104365547129789
- link LLHumerus: mass 0.0924406076207102 -> 0.0924406074551832
- link LMFemur: mass 0.123790772350432 -> 0.123790820508356
- link LMHumerus: mass 0.138065752290352 -> 0.138065758700322
- link LPalm: mass 0.071951528369027 -> 0.0719515309236498
- link LRFingerU: mass 0.0104365547041236 -> 0.0104365547129789
- link LRadius: mass 0.225239465270569 -> 0.22523946527057
- link LTibia: mass 0.197322298421 -> 0.197322267255763
- link LToe: mass 0.0300993469546569 -> 0.0300993648154242
- link LUFemur: mass 0.0588371617721 -> 0.0588371608328871
- link LUHumerus: mass 0.0562874209462877 -> 0.0562874205713043
- link LWrist: mass 0.0707291405501728 -> 0.0707291421737037
- link RFoot: mass 0.0576266868508423 -> 0.0576266868508424
- link RLFemur: mass 0.0813766060772551 -> 0.0813765868175624
- link RLFingerL: mass 0.00367689699109765 -> 0.00367689699109764
- link RLFingerU: mass 0.0104365547181582 -> 0.0104365547129788
- link RLHumerus: mass 0.092440609285167 -> 0.0924406074551833
- link RMFemur: mass 0.123790727728343 -> 0.123790820508356
- link RMHumerus: mass 0.13806574130706 -> 0.138065758700322
- link RPalm: mass 0.0719515165156188 -> 0.0719515309236498
- link RRFingerU: mass 0.0104365547185436 -> 0.0104365547129789
- link RTibia: mass 0.197322298408282 -> 0.197322267255763
- link RToe: mass 0.0300993381405375 -> 0.0300993648154242
- link RUFemur: mass 0.0588371599148218 -> 0.058837160832887
- link RUHumerus: mass 0.0562874211047921 -> 0.0562874205713042
- link RWrist: mass 0.0707291283778046 -> 0.0707291421737036
Joints:
- joint LAnkle: origin xyz=0 -0.137327472527473 0 rpy=-1.5707963267949 -1.48050713192401 1.5707963267949 -> xyz=0 -0.139941334255675 -0.0226097095250998 rpy=1.57079623659819 -1.41061489038498 -1.57079623775286
- joint LElbow1: origin xyz=0 -0.0607173844560569 0 rpy=-3.14159265358979 -0.0239343941798154 3.14159265358979 -> xyz=0 -0.0606510810810811 0 rpy=0 0 3.14159265358979
- joint LElbow2: origin xyz=0 -0.07695748040881 0 rpy=-3.03329101627937 0 -3.14159265358979 -> xyz=0 0.077023783783784 0 rpy=0 0 3.14159265358979
- joint LHip1: origin xyz=0.03048 0.0787364118309958 0.0381 rpy=-1.6707324107769 0 -1.5707963267949 -> xyz=0.03048 0.0787364118309958 0.0381 rpy=-1.5707963267949 0 -1.5707963267949
- joint LHip2: origin xyz=-0.0226409652141425 0.0437018699604634 0.00885299170630801 rpy=-0.199631486527388 -0.00987173434951005 3.09284097456322 -> xyz=-0.0226409652141426 0.0445895604395605 0 rpy=0 0 3.14159265358979
- joint LKnee1: origin xyz=-0.250689445253999 -0.0779374608440729 0.210317560896771 rpy=0 -0.21670904669546 0 -> xyz=0 -0.0684543956043956 0 rpy=0 0 0
- joint LKnee2: origin xyz=0.1790209512322 -0.0449455061888935 -0.259300751969874 rpy=0.527580516456534 0 0 -> xyz=0 -0.05 0 rpy=-0.160181436409911 0 0
- joint LLKnuckleL: origin xyz=-0.0230295534577176 0.00418692684763539 0.00654490271930316 rpy=0 0 -1.39256651875685 -> xyz=-0.03302 0 -0.00919360057874935 rpy=0 0 -1.5707963267949
- joint LLKnuckleU: origin xyz=1.84275573584247E-05 -0.0513442857142855 0 rpy=0 0 0.0795874815148373 -> xyz=0 -0.0513442857142857 0.00172665186080059 rpy=0 0 0
- joint LRKnuckleL: origin xyz=-0.0330185105270897 -0.00134428488911487 0.00626872193397954 rpy=0 0 -1.33697789041426 -> xyz=-0.03302 -0.00134428571428574 0.00707292307692295 rpy=0 0 -1.5707963267949
- joint LRKnuckleU: origin xyz=1.84275573584247E-05 -0.05 0.000276180785323571 rpy=0 0 -0.00110800345436074 -> xyz=0 -0.05 0.000276794871794911 rpy=0 0 0
- joint LShoulder1: origin xyz=0.27432 0.121591734569834 0.0381 rpy=-1.59149829481724 0 -1.5707963267949 -> xyz=0.27432 0.121591734569834 0.0381 rpy=-1.57079634169606 0 -1.5707963267949
- joint LShoulder2: origin xyz=-0.0226638309978741 0.0435202378384486 0.00180293951314842 rpy=-0.0414007011337932 -0.000517705291545505 3.12909570306687 -> xyz=-0.0226638309978741 0.0435575675675675 0 rpy=0 0 3.14159265358979
- joint LToe: origin xyz=0.05000625 0 0 rpy=0 0 0.371183380985709 -> xyz=0.05000625 0 0 rpy=0 0 0
- joint LWrist1: origin xyz=0 -0.154047567567568 0 rpy=1.57079632679489 -1.56895051945567 -1.57079632679489 -> xyz=0 -0.154047567567568 0 rpy=3.14159265358979 -1.5707963267949 0
- joint LWrist2: origin xyz=0 0 0 rpy=0 -0.0666240559322892 0 -> xyz=0 0 0 rpy=0 0 0
- joint RAnkle: origin xyz=0 -0.136901508135358 -0.000553841883564526 rpy=-1.5707963267949 -1.19317274042075 1.5707963267949 -> xyz=0 -0.141756043956044 0 rpy=3.14159265358979 -1.5707963267949 0
- joint RElbow1: origin xyz=0 -0.0477044130779104 0 rpy=-3.14159265358979 -0.043289072999253 3.14159265358979 -> xyz=0 -0.0606510810810811 0 rpy=0 0 3.14159265358979
- joint RElbow2: origin xyz=0 -0.0899704517869562 0 rpy=0.441432869104159 0 0 -> xyz=0 0.0770237837837839 0 rpy=0 0 0
- joint RHip1: origin xyz=0.03048 -0.0787364118309958 0.0380999999999998 rpy=-1.76467257912073 0 -1.5707963267949 -> xyz=0.03048 -0.0787364118309958 0.0381 rpy=1.5707963267949 0 -1.57079634169606
- joint RHip2: origin xyz=0.0226409652141427 0.0412792847511113 0.0168597019733423 rpy=-0.386092293810914 -0.0367782603560909 3.05138185304591 -> xyz=0.0226409652141425 -0.0445895604395604 0 rpy=3.14159265358979 0 3.14159265358979
- joint RKnee1: origin xyz=0 -0.073581670471731 0 rpy=0 -0.221518435550964 0 -> xyz=0 -0.0684543956043956 0 rpy=0 0 0
- joint RKnee2: origin xyz=0 -0.05 0 rpy=0.915177643816393 0 0 -> xyz=0 -0.05 0 rpy=0 0 0
- joint RLKnuckleL: origin xyz=-0.0330199999999999 0 -0.00815796517422882 rpy=0 0 -1.42852646400694 -> xyz=-0.0330199999999999 -0.0013442857142858 -0.00774374358974361 rpy=0 0 -1.5707963267949
- joint RLKnuckleU: origin xyz=0 -0.0513442857142855 0.000962687485064811 rpy=0 0 0.0322968189623831 -> xyz=0 -0.05 0.000276794871794883 rpy=0 0 0
- joint RRKnuckleL: origin xyz=-0.0329799188990406 -0.00134368805419179 0.00680985742226439 rpy=0 0 -1.42676533867921 -> xyz=-0.0330199999999999 -0.00134428571428585 0.007072923076923 rpy=0 0 -1.5707963267949
- joint RRKnuckleU: origin xyz=0 -0.05 0.000276725129630978 rpy=0 0 -0.0298203287563768 -> xyz=0 -0.05 0.000276794871794883 rpy=0 0 0
- joint RShoulder1: origin xyz=0.27432 -0.121591734569834 0.0381 rpy=-1.83631660924277 0 -1.5707963267949 -> xyz=0.27432 -0.121591734569834 0.0381 rpy=-1.5707963267949 0 -1.5707963267949
- joint RShoulder2: origin xyz=0.0226638309978741 0.0435575675675675 0 rpy=0 0 -3.1129739297594 -> xyz=0.0226638309978741 0.0435575675675675 0 rpy=0 0 3.14159265358979
- joint RToe: origin xyz=0.05000625 0 0 rpy=0 0 -0.000476651083853421 -> xyz=0.05000625 0 0 rpy=0 0 0
- joint RWrist1: origin xyz=0 -0.154047567567566 0 rpy=-1.5707963267949 0.763601167462532 -1.5707963267949 -> xyz=0 0.154047567567568 0 rpy=0 -1.5707963267949 0
- joint RWrist2: origin xyz=0 0 0 rpy=0 -0.0224487832351522 0 -> xyz=0 0 0 rpy=0 0 0

Commit message: Fixed weird urdf error (hopefully)

File: v1/urdf/v1.urdf (robot description, URDF)
Before this commit: robot v1, 33 links, 32 joints
Links:
- removed link LFoot
- removed link LLFingerL
- removed link LLFingerU
- removed link LRFingerL
- removed link LRFingerU
- removed link RFoot
- removed link RLFingerL
- removed link RLFingerU
- removed link RRFingerL
- removed link RRFingerU
- added link LHeel, mass 0.0576266868508424; collision mesh filename=package://v1/meshes/LHeel.STL; visual mesh filename=package://v1/meshes/LHeel.STL
- added link LLFinger1, mass 0.0104365547129789; collision mesh filename=package://v1/meshes/LLFinger1.STL; visual mesh filename=package://v1/meshes/LLFinger1.STL
- added link LLFinger2, mass 0.00367689699109764; collision mesh filename=package://v1/meshes/LLFinger2.STL; visual mesh filename=package://v1/meshes/LLFinger2.STL
- added link LRFinger1, mass 0.0104365547129789; collision mesh filename=package://v1/meshes/LRFinger1.STL; visual mesh filename=package://v1/meshes/LRFinger1.STL
- added link LRFinger2, mass 0.00367689699109764; collision mesh filename=package://v1/meshes/LRFinger2.STL; visual mesh filename=package://v1/meshes/LRFinger2.STL
- added link RHeel, mass 0.0576266868508424; collision mesh filename=package://v1/meshes/RHeel.STL; visual mesh filename=package://v1/meshes/RHeel.STL
- added link RLFinger1, mass 0.0104365547129788; collision mesh filename=package://v1/meshes/RLFinger1.STL; visual mesh filename=package://v1/meshes/RLFinger1.STL
- added link RLFinger2, mass 0.00367689699109764; collision mesh filename=package://v1/meshes/RLFinger2.STL; visual mesh filename=package://v1/meshes/RLFinger2.STL
- added link RRFInger2, mass 0.00367689699109764; collision mesh filename=package://v1/meshes/RRFInger2.STL; visual mesh filename=package://v1/meshes/RRFInger2.STL
- added link RRFinger1, mass 0.0104365547129789; collision mesh filename=package://v1/meshes/RRFinger1.STL; visual mesh filename=package://v1/meshes/RRFinger1.STL
- link LPalm: mass 0.0719515309236498 -> 0.0490148886446744
- link LWrist: mass 0.0707291421737037 -> 0.0217142535290293
- link RLHumerus: mass 0.0924406074551833 -> 0.0924406074551832
- link RPalm: mass 0.0719515309236498 -> 0.0490148886446744
- link RWrist: mass 0.0707291421737036 -> 0.0217142535290293
Joints:
- removed joint LLKnuckleL
- removed joint LLKnuckleU
- removed joint LRKnuckleL
- removed joint LRKnuckleU
- removed joint RLKnuckleL
- removed joint RLKnuckleU
- removed joint RRKnuckleL
- removed joint RRKnuckleU
- added joint LLKnuckle1: type continuous, parent LPalm, child LLFinger1, origin xyz=0 -0.0368299999999999 0.00144985698900568 rpy=0 0 0, axis 0 0 1
- added joint LLKnuckle2: type continuous, parent LLFinger1, child LLFinger2, origin xyz=-0.03302 0 -0.00919360057874935 rpy=0 0 -1.5707963267949, axis 0 0 1
- added joint LRKnuckle1: type continuous, parent LPalm, child LRFinger1, origin xyz=0 -0.0368299999999999 0.00144985698900568 rpy=0 0 0, axis 0 0 1
- added joint LRKnuckle2: type continuous, parent LRFinger1, child LRFinger2, origin xyz=-0.03302 0 0.00562306608791727 rpy=0 0 -1.5707963267949, axis 0 0 1
- added joint RLKnuckle1: type continuous, parent RPalm, child RLFinger1, origin xyz=0 -0.0368300000000001 0.00144985698900574 rpy=0 0 0, axis 0 0 1
- added joint RLKnuckle2: type continuous, parent RLFinger1, child RLFinger2, origin xyz=-0.0330199999999999 0 -0.00919360057874935 rpy=0 0 -1.5707963267949, axis 0 0 1
- added joint RRKnuckle1: type continuous, parent RPalm, child RRFinger1, origin xyz=0 -0.0368300000000001 0.00144985698900574 rpy=0 0 0, axis 0 0 1
- added joint RRKnuckle2: type continuous, parent RRFinger1, child RRFInger2, origin xyz=-0.0330199999999999 0 0.00562306608791727 rpy=0 0 -1.5707963267949, axis 0 0 1
- joint LAnkle: child LFoot -> LHeel; origin xyz=0 -0.139941334255675 -0.0226097095250998 rpy=1.57079623659819 -1.41061489038498 -1.57079623775286 -> xyz=0 -0.135569455799804 -0.0219033642376833 rpy=1.57079623659819 -1.41061489038498 -1.57079623775286
- joint LKnee2: origin xyz=0 -0.05 0 rpy=-0.160181436409911 0 0 -> xyz=0 -0.0544285714285714 0 rpy=-0.160181436409911 0 0
- joint LToe: parent LFoot -> LHeel
- joint LWrist2: origin xyz=0 0 0 rpy=0 0 0 -> xyz=0 -0.0145142857142858 0.000276794871794911 rpy=0 0 0
- joint RAnkle: child RFoot -> RHeel; origin xyz=0 -0.141756043956044 0 rpy=3.14159265358979 -1.5707963267949 0 -> xyz=0 -0.137327472527473 0 rpy=3.14159265358979 -1.5707963267949 0
- joint RKnee2: origin xyz=0 -0.05 0 rpy=0 0 0 -> xyz=0 -0.0544285714285715 0 rpy=0 0 0
- joint RToe: parent RFoot -> RHeel
- joint RWrist2: origin xyz=0 0 0 rpy=0 0 0 -> xyz=0 -0.0145142857142857 0.000276794871794883 rpy=0 0 0
